Commit message: Added Nav2 and AMCL

File: desc/lidar.xacro (robot description, xacro)
@@ -33,5 +33,5 @@
         <sensor name="laser" type="ray">
             <pose> 0 0 0 0 0 0 </pose>
-            <visualize>true</visualize>
+            <visualize>false</visualize>
             <update_rate>10</update_rate>
             <ray>

File: desc/robot_core.xacro (robot description, xacro)
@@ -33,4 +33,11 @@
     <!-- BASE LINK -->
     <link name="base_link">
+    </link>
+    <joint name="base_footprint_joint" type="fixed">
+        <parent link="base_link"/>
+        <child link="base_footprint"/>
+        <origin xyz="0 0 0" rpy="0 0 0"/>
+    </joint>
+    <link name="base_footprint">
     </link>
     <!-- CHASSIS LINK -->
